File: PIC32 Dev Board/PIC32 Dev Board.kicad_sch (KiCad schematic)
At the start: 16 parts, among them J1 Barrel_Jack, SW1 SW_Push, U1 PIC32MX575F256H, U2 AMS1117-3.3, Y1 8MHz

Commit message: Add files via upload
Parts:
- added C16, C18: 10uF, symbol Device:C
- added C6: 0.1uF, symbol Device:C
- added C7: 4.7uF, symbol Device:C
- added D1, D2, D3, D4, D5: LED, symbol Device:LED
- added FB1: 600@100MHz, symbol Device:FerriteBead
- added J2: Conn_02x03_Odd_Even, symbol Connector_Generic:Conn_02x03_Odd_Even
- added J3: USB_Micro, symbol Connector:USB_B_Micro
- added J4: Conn_02x06_Odd_Even, symbol Connector_Generic:Conn_02x06_Odd_Even
- added JP1: Conn_01x03, symbol Connector_Generic:Conn_01x03
- added R10, R11, R12, R8, R9: 470, symbol Device:R
- added R13, R14: 10k, symbol Device:R
- added R3, R4: 100, symbol Device:R
- added R5, R6: 27R, symbol Device:R
- added R7: 100k, symbol Device:R
- added SW2, SW3: SW_Push, symbol Switch:SW_Push
- added U3: USBLC6-2SC6, Package_TO_SOT_SMD:SOT-23-6, symbol Power_Protection:USBLC6-2SC6
Connections:
- net +3.3V: now also FB1.1, J2.2 (Pin_2), JP1.1 (Pin_1), R13.1, R14.1, R8.1, U3.4 (I/O2)
- net GND: now also U1.20 (AVSS), U1.25 (VSS), U1.41 (VSS), U1.9 (VSS), C16.2, C18.1, C6.1, C7.2, D1.1 (K), D2.1 (K), D3.1 (K), D4.1 (K), D5.1 (K), J2.3 (Pin_3), J3.5 (GND), J3.6 (Shield), R7.2, SW2.2, SW3.2, U3.2 (GND)
- net MCLR: now also J2.1 (Pin_1)
- net PGEC1: now reaches U1.13 (RB3)
- net PGEC1: now also R4.1
- net PGED1: now reaches U1.14 (RB2)
- net PGED1: now also R3.1
- net at U1.19 (AVDD): now also C18.2, C6.2, FB1.2
- net at C9.1: now also U1.56 (VCAP); no longer U1.20 (AVSS)
- net USB_ID: now reaches U1.33 (RF3)
- net USB_ID: now also J3.4 (ID), R7.1
- net VBUS: now reaches U1.34 (VBUS)
- net VBUS: now also C16.1, J3.1 (VBUS)
- net at U1.35 (VUSB): now also C7.1
- net USB_DM: now reaches U1.36 (RG3)
- net USB_DM: now also R6.2
- net USB_DP: now reaches U1.37 (RG2)
- net USB_DP: now also R5.2
- net RG6: now reaches U1.4 (RG6)
- net RG6: now also R9.1
- net BUT_0: now reaches U1.42 (RD8)
- net BUT_0: now also R13.2, SW2.1
- net BUT_1: now reaches U1.43 (RD9)
- net RG7: now reaches U1.5 (RG7)
- net RG7: now also R10.1
- net RG8: now reaches U1.6 (RG8)
- net RG8: now also R11.1
- net RG9: now reaches U1.8 (RG9)
- net RG9: now also R12.1
- new net: J2.5 (Pin_5), R4.2
- new net: D2.2 (A), R12.2
- new net: D5.2 (A), R9.2
- new net: R6.1, U3.5 (VBUS)
- new net: J2.4 (Pin_4), R3.2
- new net: D3.2 (A), R11.2
- new net: R5.1, U3.6 (I/O1)
- new net: J3.3 (D+), U3.1 (I/O1)
- new net: J3.2 (D-), U3.3 (I/O2)
- new net: R14.2, SW3.1
- new net: D4.2 (A), R10.2
- new net: D1.2 (A), R8.2
Other:
- note added: "BLOCK 10 : USER LEDS"
- note added: "BLOCK 11 : USER BUTTONS"
- note added: "BLOCK 12 : GPIO HEADER ACCESS - PORT B"
- note added: "BLOCK 7 : USB INTERFACE"
- note added: "BLOCK 9 : POWER LED INDICATOR"
- note removed: "BLOCK 2 : INTERNAL VOLTAGE REGULATOR (VCAP)"
- moved on the sheet: C1, C10, C11, C12, C2, C3, C4, C9, J1, R1, R2, SW1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

Commit message: Add files via upload
Parts:
- removed J4: Conn_02x06_Odd_Even, symbol Connector_Generic:Conn_02x06_Odd_Even
- added J4: Conn_02x20_Odd_Even, symbol Connector_Generic:Conn_02x20_Odd_Even
Connections:
- net +3.3V: now also J4.1 (Pin_1), J4.2 (Pin_2), J4.20 (Pin_20), J4.39 (Pin_39)
- net GND: now also J4.19 (Pin_19), J4.3 (Pin_3), J4.4 (Pin_4), J4.40 (Pin_40)
- net RB5: now reaches U1.11 (RB5)
- net RB5: now also J4.8 (Pin_8)
- net RB4: now reaches U1.12 (RB4)
- net RB4: now also J4.7 (Pin_7)
- net RB1: now reaches U1.15 (RB1)
- net RB1: now also J4.6 (Pin_6)
- net RB0: now reaches U1.16 (RB0)
- net RB0: now also J4.5 (Pin_5)
- net RB6: now reaches U1.17 (RB6)
- net RB6: now also J4.9 (Pin_9)
- net RB7: now reaches U1.18 (RB7)
- net RB7: now also J4.10 (Pin_10)
- net RB8: now reaches U1.21 (RB8)
- net RB8: now also J4.11 (Pin_11)
- net RB9: now reaches U1.22 (RB9)
- net RB9: now also J4.12 (Pin_12)
- net RB10: now reaches U1.23 (RB10)
- net RB10: now also J4.13 (Pin_13)
- net RB11: now reaches U1.24 (RB11)
- net RB11: now also J4.14 (Pin_14)
- net RB12: now reaches U1.27 (RB12)
- net RB12: now also J4.15 (Pin_15)
- net RB13: now reaches U1.28 (RB13)
- net RB13: now also J4.16 (Pin_16)
- net RB14: now reaches U1.29 (RB14)
- net RB14: now also J4.17 (Pin_17)
- net RB15: now reaches U1.30 (RB15)
- net RB15: now also J4.18 (Pin_18)
- new net RD2: J4.21 (Pin_21)
- new net RD3: J4.22 (Pin_22)
- new net RD4: J4.23 (Pin_23)
- new net RD5: J4.24 (Pin_24)
- new net RD6: J4.25 (Pin_25)
- new net RD7: J4.26 (Pin_26)
- new net RD8: J4.27 (Pin_27)
- new net RD9: J4.28 (Pin_28)
- new net RE0: J4.29 (Pin_29)
- new net RE1: J4.30 (Pin_30)
- new net RE2: J4.31 (Pin_31)
- new net RE3: J4.32 (Pin_32)
- new net RE4: J4.33 (Pin_33)
- new net RE5: J4.34 (Pin_34)
- new net RE6: J4.35 (Pin_35)
- new net RE7: J4.36 (Pin_36)
- new net RF0: J4.37 (Pin_37)
- new net RF1: J4.38 (Pin_38)
Other:
- note added: "MAIN GPIO HEADER (2x20)"
- note removed: "BLOCK 12 : GPIO HEADER ACCESS - PORT B"
